Commit message: Fixed a bug in urdf files ( and some other minor changes)
New Dynamic have NOT been generated

File: urdf/cassie.urdf (robot description, URDF)
Before this commit: robot cassie, 17 links, 16 joints
Joints:
- joint hip_rotation_left: axis 1 0 0 -> -1 0 0
- joint hip_rotation_right: axis 1 0 0 -> -1 0 0

File: urdf/cassie.xacro (robot description, xacro)
@@ -16,5 +16,5 @@
   <xacro:pelvis_abduction side="left" cname="light_grey" color="${light_grey_RGB}" stl_ext=""/>
   <xacro:pelvis_rotation side="left" cname="light_grey" color="${light_grey_RGB}" stl_ext="" reflect="1" />
-  <xacro:hip side="left" cname="light_grey" color="${light_grey_RGB}" stl_ext="" reflect="1"/>
+  <xacro:hip side="left" cname="light_grey" color="${light_grey_RGB}" stl_ext="" />
   <xacro:thigh side="left" cname="light_grey" color="${light_grey_RGB}" stl_ext="" reflect="1"/>
   <xacro:knee side="left" cname="grey" color="${grey_RGB}" stl_ext="" reflect="1"/>
@@ -24,5 +24,5 @@
   <xacro:pelvis_abduction side="right" cname="light_grey" color="${light_grey_RGB}" stl_ext="_mirror"/>
   <xacro:pelvis_rotation side="right" cname="light_grey" color="${light_grey_RGB}" stl_ext="_mirror" reflect="-1"/>
-  <xacro:hip side="right" cname="light_grey" color="${light_grey_RGB}" stl_ext="_mirror" reflect="-1"/>
+  <xacro:hip side="right" cname="light_grey" color="${light_grey_RGB}" stl_ext="_mirror"/>
   <xacro:thigh side="right" cname="light_grey" color="${light_grey_RGB}" stl_ext="_mirror" reflect="-1"/>
   <xacro:knee side="right" cname="grey" color="${grey_RGB}" stl_ext="_mirror" reflect="-1"/>
@@ -113,10 +113,10 @@
     </link>
   </xacro:macro>
-  <xacro:macro name="hip" params="side cname color stl_ext reflect">
+  <xacro:macro name="hip" params="side cname color stl_ext">
     <link name="${side}_hip">
       <inertial>
         <origin xyz="-.0557 0 0" rpy="0 0 0"/>
         <mass value="1.17" />
-        <inertia ixx=".000842" ixy=".000000246" ixz="${reflect*-.000000625}" iyy=".006080" iyz="${reflect*-.00000004}" izz=".006440" />
+        <inertia ixx=".000842" ixy=".000000246" ixz="-.000000625" iyy=".006080" iyz="-.00000004" izz=".006440" />
       </inertial>
       <visual>
@@ -248,5 +248,5 @@
     <joint name="hip_rotation_${side}" type="continuous">
       <origin xyz="0 0 -0.09" rpy="0 ${pi/2} ${-pi/2}"/>
-      <axis xyz="1 0 0"/>
+      <axis xyz="-1 0 0"/>
       <parent link="${side}_pelvis_rotation" />
       <child link="${side}_hip" />
